File: schema/trigger/trigger.kicad_sch (KiCad schematic)
At the start: 39 parts, among them IC1 RP2040_ZERO, J1 Conn_01x06_Socket, J2 Conn_01x05_Pin, J4 Conn_01x04_Pin, Q1 DMG4800LK3-13, SW1 SW_Push

Commit message: bom and some finetuning while first assembly
Parts:
- D1: value LED_Small -> LED_RED
- D2: value LED_Small -> LED_GREEN
- IC2: value ~ -> 5V0 step down
- R4: value 860k -> 1M0
