File: schema/motor/motor.kicad_pcb (KiCad board)
At the start: 2 copper layers, 50 x 50 mm, 45 parts, among them IC1 RP2040_ZERO, IC2 +5V REG, J1 Conn_01x06, J2 Conn_02x04_Odd_Even, J4 Conn_01x04_Pin, Q1 DMG4800LK3-13

Commit message: chicken squasher hw v1.0 - final touch, fabrication
Routing:
- net GND: track 14.0 -> 23.1 mm, vias 28 -> 41
Other:
- board text added: "GND"
- board text added: "VIN"
